File: pcb_test/connecteurs.kicad_sch (KiCad schematic)
At the start: 4 parts, among them J1 USB_C_Receptacle_USB2.0_14P, U2 USBLC6-2P6

Commit message: refait alimentation, changement MCU, separation schema eMMC/octospi, reajout RF
Parts:
- R1, R2: symbol Device:R -> Device:R_US
Connections:
- net +5V: no longer J1.A4 (VBUS), J1.A9 (VBUS), J1.B4 (VBUS), J1.B9 (VBUS)
- new net +5V_IN2: J1.A4 (VBUS), J1.A9 (VBUS), J1.B4 (VBUS), J1.B9 (VBUS)
Changed lines of the file:
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@@
 	(wire
 		(pts
-			(xy 46.99 24.13) (xy 48.26 24.13)
+			(xy 46.99 24.13) (xy 50.8 24.13)
 		)
 		(stroke
@@
 	(wire
 		(pts
-			(xy 48.26 22.86) (xy 48.26 24.13)
+			(xy 50.8 22.86) (xy 50.8 24.13)
 		)
 		(stroke
@@
 	)
 	(symbol
-		(lib_id "Device:R")
+		(lib_id "Device:R_US")
 		(at 53.34 31.75 90)
 		(unit 1)
@@
 		)
 		(property "Footprint" ""
-			(at 53.34 33.528 90)
+			(at 53.594 30.734 90)
 			(hide yes)
 			(show_name no)
@@
 			)
 		)
-		(property "Description" "Resistor"
+		(property "Description" "Resistor, US symbol"
 			(at 53.34 31.75 0)
 			(hide yes)
@@
 	)
 	(symbol
-		(lib_id "Device:R")
+		(lib_id "Device:R_US")
 		(at 58.42 29.21 90)
 		(unit 1)
@@
 		)
 		(property "Footprint" ""
-			(at 58.42 30.988 90)
+			(at 58.674 28.194 90)
 			(hide yes)
 			(show_name no)
@@
 			)
 		)
-		(property "Description" "Resistor"
+		(property "Description" "Resistor, US symbol"
 			(at 58.42 29.21 0)
 			(hide yes)
@@
 	(symbol
 		(lib_id "power:+5V")
-		(at 48.26 22.86 0)
+		(at 50.8 22.86 0)
 		(unit 1)
 		(body_style 1)
@@
 		(fields_autoplaced yes)
 		(property "Reference" "#PWR01"
-			(at 48.26 26.67 0)
-			(hide yes)
-			(show_name no)
-			(do_not_autoplace no)
-			(effects
-				(font
-					(size 1.27 1.27)
-				)
-			)
-		)
-		(property "Value" "+5V"
-			(at 48.26 17.78 0)
+			(at 50.8 26.67 0)
+			(hide yes)
+			(show_name no)
+			(do_not_autoplace no)
+			(effects
+				(font
+					(size 1.27 1.27)
+				)
+			)
+		)
+		(property "Value" "+5V_IN2"
+			(at 50.8 17.78 0)
 			(show_name no)
 			(do_not_autoplace no)
@@
 		)
 		(property "Footprint" ""
-			(at 48.26 22.86 0)
+			(at 50.8 22.86 0)
 			(hide yes)
 			(show_name no)
@@
 		)
 		(property "Datasheet" ""
-			(at 48.26 22.86 0)
+			(at 50.8 22.86 0)
 			(hide yes)
 			(show_name no)
@@
 		)
 		(property "Description" "Power symbol creates a global label with name \"+5V\""
-			(at 48.26 22.86 0)
-			(hide yes)
-			(show_name no)
+			(at 50.8 22.86 0)
+			(hide yes)
+			(show_name no)
