File: pcb_test/octospi.kicad_sch (KiCad schematic)
At the start: 34 parts, among them U7 MX66LM1G45GXDI00

Commit message: alimentation finale. Retouches testpoints et condo decouplage, finalisation requis, ajout sheet finale.
Parts:
- removed C29, C31, C33: 1u, symbol Device:C
Other:
- moved on the sheet: C32, C34
