File: pcb_test/telecom.kicad_sch (KiCad schematic)
At the start: 0 parts

Commit message: alimentation finale. Retouches testpoints et condo decouplage, finalisation requis, ajout sheet finale.
Other:
- note added: "SI4464"
Changed lines of the file:
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@@
 	(generator_version "10.0")
 	(paper "A4")
+	(text "SI4464"
+		(exclude_from_sim no)
+		(at 107.9019 63.4843 0)
+		(effects
+			(font
+				(size 1.27 1.27)
+			)
+			(justify left)
+		)
+	)
 )
