File: pcb_test/Ethernet.kicad_sch (KiCad schematic)
At the start: 1 part, among them U16 LAN8742A

Commit message: Presque fini i guess
Parts:
- added C33, C46, C58: 0.1u, symbol Device:C
- added C59: 0.47u, symbol Device:C
- added C60: 1u, symbol Device:C
- added C61, C68: 4.7u, symbol Device:C
- added C62: 22n, symbol Device:C
- added C63, C64, C65, C66: 10p, symbol Device:C
- added C93, C94: 13p, symbol Device:C
- added FB1: FerriteBead, symbol Device:FerriteBead
- added J2: RJ45_Amphenol_RJMG1BD3B8K1ANR, Connector_RJ:RJ45_Amphenol_54602-x08_Horizontal, symbol Connector:RJ45_Amphenol_RJMG1BD3B8K1ANR
- added R103, R104, R110, R115, R116, R117, R118, R119, R120, R122, R124, R125, R126, R127, R129, R130, R132, R133: 0, symbol Device:R_US
- added R105, R106: 33R, symbol Device:R_US
- added R108, R121, R136, R137, R138: 10k, symbol Device:R_US
- added R109: 12.1k, symbol Device:R_US
- added R111, R112, R113, R114: 49.9R, symbol Device:R_US
- added R123, R128, R131, R134: 270, symbol Device:R_US
- added Y2: ABM8-25.000MHZ-D1X-T, Crystal:Crystal_SMD_Abracon_ABM8G-4Pin_3.2x2.5mm, symbol Device:Crystal_GND24
Connections:
- net at U16.1 (VDD2A): now also U16.19 (VDD1A), R103.2
- net RXER/PHYAD0: now reaches U16.10 (RXER/PHYAD0)
- net RXER/PHYAD0: now also R119.2, R120.1
- net ETH_RMII_CRS_DV: now reaches U16.11 (CRS_DV/MODE2)
- net ETH_RMII_CRS_DV: now also R121.2, R122.1
- net ETH_MDIO: now reaches U16.12 (MDIO)
- net ETH_MDIO: now also R108.2
- net ETH_MDC: now reaches U16.13 (MDC)
- net ETH_RMII_REFCLK: now reaches U16.14 (~{INT}/REFCLKO)
- net ETH_RMII_REFCLK: now also R138.2
- net ~{RST}: now reaches U16.15 (~{RST})
- net ETH_RMII_TXEN: now reaches U16.16 (TXEN)
- net ETH_RMII_TXD0: now reaches U16.17 (TXD0)
- net ETH_RMII_TXD1: now reaches U16.18 (TXD1)
- net LED2/~{INTSEL}: now reaches U16.2 (LED2/~{INTSEL})
- net LED2/~{INTSEL}: now also R127.2, R132.1
- net at U16.20 (TXN): now also C65.1, J2.R2 (TD-), R113.2
- net at U16.21 (TXP): now also C66.1, J2.R1 (TD+), R110.2, R114.2
- net at U16.22 (RXN): now also C62.1, C63.1, J2.R6 (RD-), R111.2
- net at U16.23 (RXP): now also C64.1, J2.R3 (RD+), R112.2
- net at U16.24 (RBIAS): now also R109.1
- net GND: now reaches U16.25 (VSS)
- net GND: now also C33.2, C46.2, C58.2, C59.2, C60.2, C61.2, C62.2, C63.2, C64.2, C65.2, C66.2, C68.2, C93.2, C94.2, J2.R8, J2.SH, R109.2, R115.2, R118.2, R120.2, R122.2, R130.2, R133.2, Y2.2 (G), Y2.4 (G)
- net LED1/REGOFF: now reaches U16.3 (LED1/REGOFF)
- net LED1/REGOFF: now also R125.2, R129.1
- net XTAL2: now reaches U16.4 (XTAL2)
- net XTAL2: now also C94.1, Y2.3
- net XTAL1: now reaches U16.5 (XTAL1/CLKIN)
- net XTAL1: now also C93.1, Y2.1
- net VDDCR: now reaches U16.6 (VDDCR)
- net VDDCR: now also C59.1, C60.1, C61.1
- net RXD1/MODE1: now reaches U16.7 (RXD1/MODE1)
- net RXD1/MODE1: now also R106.2, R117.2, R118.1, R137.2
- net RXD0/MODE0: now reaches U16.8 (RXD0/MODE0)
- net RXD0/MODE0: now also R105.2, R115.1, R116.2, R136.2
- net at U16.9 (VDDIO): now also R104.2
- new net: R123.1, R124.2, R125.1
- new net: R126.2, R127.1, R128.1
- new net: R129.2, R130.1, R131.1
- new net: R132.2, R133.1, R134.1
- new net: J2.R4 (TCT), J2.R5 (RCT)
- new net +3V3: C33.1, FB1.1, R104.1, R108.1, R116.1, R117.1, R119.1, R121.1, R124.1, R126.1, R136.1, R137.1, R138.1
- new net +3V3A: C46.1, C58.1, C68.1, FB1.2, R103.1, R110.1, R111.1, R112.1, R113.1, R114.1
- new net ETH_RMII_RXD0: R105.1
- new net ETH_RMII_RXD1: R106.1
- new net LED_G_ANODE: J2.L4, R128.2
- new net LED_G_CATHODE: J2.L3, R134.2
- new net LED_Y_ANODE: J2.L1, R123.2
- new net LED_Y_CATHODE: J2.L2, R131.2
Other:
- moved on the sheet: U16
