File: pcb_test/buzzer.kicad_sch (KiCad schematic)
At the start: 0 parts

Commit message: Presque fini i guess
Parts:
- added C10, C12: 0.1u, symbol Device:C
- added C29: 8n, symbol Device:C
- added C31: 22n, symbol Device:C
- added LS1: Speaker, symbol Device:Speaker
- added R100: 1k, symbol Device:R_US
- added R101: 20k, symbol Device:R_US
- added R102: 15k, symbol Device:R_US
- added U19: (no value), Package_SO:SOIC-8_3.9x4.9mm_P1.27mm, symbol stuff:LM4818
Connections:
- new net: R101.2, R102.1, U19.4 (IN-)
- new net: LS1.1, R102.2, U19.8 (OUT+)
- new net: LS1.2, U19.5 (OUT-)
- new net: C31.2, R101.1
- new net: C29.1, C31.1, R100.2
- new net +5V: C10.1, U19.6 (Vcc)
- new net BUZZER_EN: U19.1 (SDB)
- new net BUZZER_SIG: R100.1
- new net GND: C10.2, C12.2, C29.2, U19.7 (GND)
- new net byp: C12.1, U19.2 (BYPASS), U19.3 (IN+)
Other:
- note added: "Amplifier should output ~250 mW into 8 ohms load."
- note added: "Speaker"
- note added: "Speaker amplifier circuit"
- note added: "Speaker amplifier power & logic"
- note added: "Speaker impedance is 8 ohms"
