File: pcb_test/pcb_test.kicad_sch (KiCad schematic)
At the start: 1 part, among them U1 STM32U5G9ZJJxQ

Commit message: Ajout testpoints
Parts:
- U1: footprint Package_BGA:UFBGA-144_10x10mm_Layout12x12_P0.8mm -> Package_QFP:LQFP-144_20x20mm_P0.5mm

Commit message: refait alimentation, changement MCU, separation schema eMMC/octospi, reajout RF
Parts:
- removed U1: STM32U5G9ZJJxQ, Package_QFP:LQFP-144_20x20mm_P0.5mm, symbol MCU_ST_STM32U5:STM32U5G9ZJJxQ
- added C48: 1u, symbol Device:C
- added C49: 0.1u, symbol Device:C
- added C85, C86: 7p, symbol Device:C
- added D3: LED_RGB, symbol Device:LED_RGB
- added R57, R58: 10k, symbol Device:R_US
- added R59, R60, R61: 120, symbol Device:R
- added TP65, TP66, TP68: TestPoint, symbol Connector:TestPoint
- added U13: 24LC08, Package_SO:SOIC-8_3.9x4.9mm_P1.27mm, symbol Memory_EEPROM:24LC08
- added Y1: ABM8-16.000MHZ-7-1-U-T, Crystal:Crystal_SMD_Abracon_ABM8G-4Pin_3.2x2.5mm, symbol Device:Crystal_GND24
Connections:
- new net: D3.1 (RK), R59.1
- new net: D3.2 (GK), R60.1
- new net: D3.3 (BK), R61.1
- new net +3.3V: C48.1, C49.1, R57.1, R58.1, U13.8 (VCC)
- new net EEPROM_SCL: R58.2, TP65.1, U13.6 (SCL)
- new net EEPROM_SDA: R57.2, TP66.1, U13.5 (SDA)
- new net GND: C48.2, C49.2, C85.2, C86.2, R59.2, R60.2, R61.2, TP68.1, U13.4 (GND), U13.7 (WP), Y1.2 (G), Y1.4 (G)
- new net RCC_OSC_IN: C85.1, Y1.3
- new net RCC_OSC_OUT: C86.1, Y1.1
- new net RGB_B_TIM1: D3.4 (BA)
- new net RGB_G_TIM1: D3.5 (GA)
- new net RGB_R_TIM1: D3.6 (RA)
- no-connect marks 0 -> 3
Other:
- sheet stockage renamed eMMC
- added sheet octoSPI (octospi.kicad_sch)
- note added: "8Kb EEPROM"
- note added: "RGB LEDs"
- note added: "XTAL OSCILLATOR"

Commit message: alimentation finale. Retouches testpoints et condo decouplage, finalisation requis, ajout sheet finale.
Connections:
- net RGB_B_TIM1: no longer names the net of D3.4 (BA)
- net RGB_G_TIM1: no longer names the net of D3.5 (GA)
- net RGB_R_TIM1: no longer names the net of D3.6 (RA)
Other:
- sheet alimentation renamed alimentation (done)
- sheet capteurs renamed capteurs (done)
- sheet communication renamed communication (done)
- sheet eMMC renamed eMMC (done)
- sheet gps renamed gps (done)
- sheet octoSPI renamed octoSPI (done)
- added sheet Buzzer (buzzer.kicad_sch)
- added sheet Ethernet (Ethernet.kicad_sch)
- added sheet RF (telecom.kicad_sch)
- added sheet SD card (sd_card.kicad_sch)
Changed lines of the file:
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@@
-		)
-	)
-	(global_label "RGB_B_TIM1"
-		(shape input)
-		(at 30.48 245.11 90)
-		(fields_autoplaced yes)
-		(effects
-			(font
-				(size 1.27 1.27)
-			)
-			(justify left)
-		)
-		(property "Intersheetrefs" "${INTERSHEET_REFS}"
-			(at 30.48 230.8763 90)
-			(hide yes)
-			(show_name no)
-			(do_not_autoplace no)
-			(effects
-				(font
-					(size 1.27 1.27)
-				)
-				(justify left)
-			)
-		)
-	)
-	(global_label "RGB_R_TIM1"
-		(shape input)
-		(at 20.32 245.11 90)
-		(fields_autoplaced yes)
-		(effects
-			(font
-				(size 1.27 1.27)
-			)
-			(justify left)
-		)
-		(property "Intersheetrefs" "${INTERSHEET_REFS}"
-			(at 20.32 230.8763 90)
-			(hide yes)
-			(show_name no)
-			(do_not_autoplace no)
-			(effects
-				(font
-					(size 1.27 1.27)
-				)
-				(justify left)
-			)
-		)
-	)
-	(global_label "RGB_G_TIM1"
-		(shape input)
-		(at 25.4 245.11 90)
-		(fields_autoplaced yes)
-		(effects
-			(font
-				(size 1.27 1.27)
-			)
-			(justify left)
-		)
-		(property "Intersheetrefs" "${INTERSHEET_REFS}"
-			(at 25.4 230.8763 90)
-			(hide yes)
-			(show_name no)
-			(do_not_autoplace no)
-			(effects
-				(font
-					(size 1.27 1.27)
-				)
-				(justify left)
-			)
 		)
 	)
@@
 		(in_pos_files yes)
 		(dnp no)
-		(fields_autoplaced yes)
 		(property "Reference" "Y1"
-			(at 30.48 189.23 0)
+			(at 30.48 193.04 0)
 			(show_name no)
 			(do_not_autoplace no)
@@
 		(property "Value" "ABM8-16.000MHZ-7-1-U-T"
 			(at 30.48 191.77 0)
+			(hide yes)
 			(show_name no)
 			(do_not_autoplace no)
@@
 	)
 	(sheet
-		(at 16.51 35.56)
+		(at 16.51 41.91)
 		(size 12.7 3.81)
 		(exclude_from_sim no)
@@
 			(color 0 0 0 0)
 		)
-		(property "Sheetname" "eMMC"
-			(at 16.51 34.8484 0)
+		(property "Sheetname" "eMMC (done)"
+			(at 16.51 41.1984 0)
 			(show_name no)
 			(do_not_autoplace no)
@@
 		)
 		(property "Sheetfile" "stockage.kicad_sch"
-			(at 16.51 39.9546 0)
+			(at 16.51 46.3046 0)
 			(show_name no)
 			(do_not_autoplace no)
@@
 	)
 	(sheet
-		(at 16.51 25.4)
+		(at 16.51 68.58)
 		(size 12.7 3.81)
 		(exclude_from_sim no)
@@
 			(color 0 0 0 0)
 		)
-		(property "Sheetname" "communication"
-			(at 16.51 24.6884 0)
+		(property "Sheetname" "communication (done)"
+			(at 16.51 67.8684 0)
 			(show_name no)
 			(do_not_autoplace no)
@@
 		)
 		(property "Sheetfile" "communication.kicad_sch"
-			(at 16.51 29.7946 0)
+			(at 16.51 72.9746 0)
 			(show_name no)
 			(do_not_autoplace no)
@@
 	)
 	(sheet
-		(at 16.51 66.04)
+		(at 16.51 95.25)
 		(size 12.7 3.81)
 		(exclude_from_sim no)
@@
 		)
 		(property "Sheetname" "connecteurs"
-			(at 16.51 65.3284 0)
+			(at 16.51 94.5384 0)
 			(show_name no)
 			(do_not_autoplace no)
@@
 		)
 		(property "Sheetfile" "connecteurs.kicad_sch"
-			(at 16.51 70.4346 0)
+			(at 16.51 99.6446 0)
 			(show_name no)
 			(do_not_autoplace no)
@@
 	)
 	(sheet
-		(at 16.51 74.93)
+		(at 16.51 86.36)
 		(size 12.7 3.81)
 		(exclude_from_sim no)
@@
 			(color 0 0 0 0)
 		)
-		(property "Sheetname" "octoSPI"
-			(at 16.51 74.2184 0)
+		(property "Sheetname" "RF"
+			(at 16.51 85.6484 0)
 			(show_name no)
 			(do_not_autoplace no)
@@
 			)
 		)
-		(property "Sheetfile" "octospi.kicad_sch"
-			(at 16.51 79.3246 0)
+		(property "Sheetfile" "telecom.kicad_sch"
+			(at 16.51 90.7546 0)
 			(show_name no)
 			(do_not_autoplace no)
@@
 			(project "pcb_test"
 				(path "/369fde0b-6a31-488a-9037-ea8dd8fac03b"
-					(page "8")
+					(page "9")
 				)
 			)
@@
 	)
 	(sheet
-		(at 16.51 45.72)
+		(at 16.51 24.13)
 		(size 12.7 3.81)
 		(exclude_from_sim no)
@@
 			(color 0 0 0 0)
 		)
-		(property "Sheetname" "capteurs"
-			(at 16.51 45.0084 0)
+		(property "Sheetname" "octoSPI (done)"
+			(at 16.51 23.4184 0)
 			(show_name no)
 			(do_not_autoplace no)
@@
 			)
 		)
+		(property "Sheetfile" "octospi.kicad_sch"
+			(at 16.51 28.5246 0)
+			(show_name no)
+			(do_not_autoplace no)
+			(effects
+				(font
+					(size 1.27 1.27)
+				)
+				(justify left top)
+			)
+		)
+		(instances
+			(project "pcb_test"
+				(path "/369fde0b-6a31-488a-9037-ea8dd8fac03b"
+					(page "8")
+				)
+			)
+		)
+	)
+	(sheet
+		(at 16.51 77.47)
+		(size 12.7 3.81)
+		(exclude_from_sim no)
+		(in_bom yes)
+		(on_board yes)
+		(dnp no)
+		(fields_autoplaced yes)
+		(stroke
+			(width 0.1524)
+			(type solid)
+		)
+		(fill
+			(color 0 0 0 0)
+		)
+		(property "Sheetname" "Ethernet"
+			(at 16.51 76.7584 0)
+			(show_name no)
+			(do_not_autoplace no)
+			(effects
+				(font
+					(size 1.27 1.27)
+				)
+				(justify left bottom)
+			)
+		)
+		(property "Sheetfile" "Ethernet.kicad_sch"
+			(at 16.51 81.8646 0)
+			(show_name no)
+			(do_not_autoplace no)
+			(effects
+				(font
+					(size 1.27 1.27)
+				)
+				(justify left top)
+			)
+		)
+		(instances
+			(project "pcb_test"
+				(path "/369fde0b-6a31-488a-9037-ea8dd8fac03b"
+					(page "11")
+				)
+			)
+		)
+	)
+	(sheet
+		(at 16.51 50.8)
+		(size 12.7 3.81)
+		(exclude_from_sim no)
+		(in_bom yes)
+		(on_board yes)
+		(dnp no)
+		(fields_autoplaced yes)
+		(stroke
+			(width 0.1524)
+			(type solid)
+		)
+		(fill
+			(color 0 0 0 0)
+		)
+		(property "Sheetname" "capteurs (done)"
+			(at 16.51 50.0884 0)
+			(show_name no)
+			(do_not_autoplace no)
+			(effects
+				(font
+					(size 1.27 1.27)
+				)
+				(justify left bottom)
+			)
+		)
 		(property "Sheetfile" "capteurs.kicad_sch"
-			(at 16.51 50.1146 0)
+			(at 16.51 55.1946 0)
 			(show_name no)
 			(do_not_autoplace no)
@@
 				(path "/369fde0b-6a31-488a-9037-ea8dd8fac03b"
 					(page "5")
+				)
+			)
+		)
+	)
+	(sheet
+		(at 16.51 104.14)
+		(size 12.7 3.81)
+		(exclude_from_sim no)
+		(in_bom yes)
+		(on_board yes)
+		(dnp no)
+		(fields_autoplaced yes)
+		(stroke
+			(width 0.1524)
+			(type solid)
+		)
+		(fill
+			(color 0 0 0 0)
+		)
+		(property "Sheetname" "Buzzer"
+			(at 16.51 103.4284 0)
+			(show_name no)
+			(do_not_autoplace no)
+			(effects
+				(font
+					(size 1.27 1.27)
+				)
+				(justify left bottom)
+			)
+		)
+		(property "Sheetfile" "buzzer.kicad_sch"
+			(at 16.51 108.5346 0)
+			(show_name no)
+			(do_not_autoplace no)
+			(effects
+				(font
+					(size 1.27 1.27)
+				)
+				(justify left top)
+			)
+		)
+		(instances
+			(project "pcb_test"
+				(path "/369fde0b-6a31-488a-9037-ea8dd8fac03b"
+					(page "12")
 				)
 			)
@@
 			(color 0 0 0 0)
 		)
-		(property "Sheetname" "alimentation"
+		(property "Sheetname" "alimentation (done)"
 			(at 16.51 14.5284 0)
 			(show_name no)
@@
 	)
 	(sheet
-		(at 16.51 55.88)
+		(at 16.51 59.69)
 		(size 12.7 3.81)
 		(exclude_from_sim no)
@@
 			(color 0 0 0 0)
 		)
-		(property "Sheetname" "gps"
-			(at 16.51 55.1684 0)
+		(property "Sheetname" "gps (done)"
+			(at 16.51 58.9784 0)
 			(show_name no)
 			(do_not_autoplace no)
@@
 		)
 		(property "Sheetfile" "gps.kicad_sch"
-			(at 16.51 60.2746 0)
+			(at 16.51 64.0846 0)
 			(show_name no)
 			(do_not_autoplace no)
@@
 				)
 			)
+		)
+	)
+	(sheet
+		(at 16.51 33.02)
+		(size 12.7 3.81)
+		(exclude_from_sim no)
+		(in_bom yes)
+		(on_board yes)
+		(dnp no)
+		(fields_autoplaced yes)
+		(stroke
+			(width 0.1524)
+			(type solid)
+		)
+		(fill
+			(color 0 0 0 0)
+		)
+		(property "Sheetname" "SD card"
+			(at 16.51 32.3084 0)
+			(show_name no)
+			(do_not_autoplace no)
+			(effects
+				(font
+					(size 1.27 1.27)
+				)
+				(justify left bottom)
+			)
+		)
+		(property "Sheetfile" "sd_card.kicad_sch"
+			(at 16.51 37.4146 0)
+			(show_name no)
+			(do_not_autoplace no)
+			(effects
+				(font
+					(size 1.27 1.27)
+				)
+				(justify left top)
+			)
+		)
+		(instances
+			(project "pcb_test"
+				(path "/369fde0b-6a31-488a-9037-ea8dd8fac03b"
+					(page "10")
+				)
+			)

Commit message: Presque fini i guess
Parts:
- removed C48: 1u, symbol Device:C
- removed R59, R60, R61: 120, symbol Device:R
- added C71, C72, C73, C74, C75, C76, C77, C78, C79, C80, C81, C82, C83, C84, C87, C88, C89, C90, C91, C92: 0.1u, symbol Device:C
- added Q4, Q5, Q6: 2SC5658, symbol Simulation_SPICE:NPN
- added R59, R60, R61: 50k, symbol Device:R_US
- added U20: (no value), Package_QFP:LQFP-176_24x24mm_P0.5mm, symbol stuff:STM32H5E4IK
- C85, C86: value 7p -> 13p
- Y1: value ABM8-16.000MHZ-7-1-U-T -> ABM8-25.000MHZ-D1X-T
Connections:
- net +3.3V: now also C72.1, C73.1, C74.1, C75.1, C76.1, C77.1, C78.1, C79.1, C80.1, C81.1, C82.1, C83.1, C84.1, C87.1, C88.1, C89.1, C90.1, C91.1, C92.1, U20.103 (VDD), U20.114 (VDD), U20.125 (VDDUSB), U20.127 (VDD), U20.136 (VDD), U20.149 (VDDIO2), U20.15 (VDD), U20.159 (VDD), U20.172 (VDD), U20.23 (VDD), U20.36 (VDD), U20.38 (VREF+), U20.39 (VDDA), U20.49 (VDD), U20.6 (VBAT), U20.62 (VDD), U20.72 (VDD), U20.83 (VDD), U20.91 (VDD)
- net GND: now also C71.2, C72.2, C73.2, C74.2, C75.2, C76.2, C77.2, C78.2, C79.2, C80.2, C81.2, C82.2, C83.2, C84.2, C87.2, C88.2, C89.2, C90.2, C91.2, C92.2, Q4.3 (E), Q5.3 (E), Q6.3 (E), U20.102 (VSS), U20.113 (VSS), U20.126 (VSS), U20.135 (VSS), U20.14 (VSS), U20.148 (VSS), U20.158 (VSS), U20.22 (VSS), U20.37 (VSSA), U20.48 (VSS), U20.61 (VSS), U20.71 (VSS), U20.82 (VSS)
- net at D3.1 (RK): now also Q4.1 (C)
- net at D3.2 (GK): now also Q5.1 (C)
- net at D3.3 (BK): now also Q6.1 (C)
- net +5V: now reaches D3.4 (BA)
- net +5V: now also D3.5 (GA), D3.6 (RA)
- new net: C71.1, U20.171 (VCAP), U20.81 (VCAP)
- new net: Q6.2 (B), R61.2
- new net: Q4.2 (B), R59.2
- new net: Q5.2 (B), R60.2
- new net BUZZER_EN: U20.35 (PC3)
- new net BUZZER_SIG: U20.40 (PA0)
- new net ETH_MDC: U20.33 (PC1)
- new net ETH_MDIO: U20.42 (PA2)
- new net ETH_RMII_CRS_DV: U20.53 (PA7)
- new net ETH_RMII_REFCLK: U20.41 (PA1)
- new net ETH_RMII_RXD0: U20.54 (PC4)
- new net ETH_RMII_RXD1: U20.55 (PC5)
- new net ETH_RMII_TXEN: U20.51 (PA5)
- new net LED_B: R61.1
- new net LED_G: R60.1
- new net LED_R: R59.1
Other:
- sheet Buzzer renamed Buzzer (done)
- sheet Ethernet renamed Ethernet (done)
- sheet SD card renamed SD card (done)
- removed sheet RF
- moved on the sheet: C49, D3, R57, R58, TP65, TP66, TP68, U13
