File: pcb_test/sd_card.kicad_sch (KiCad schematic)
At the start: 0 parts

Commit message: Presque fini i guess
Parts:
- added C56, C57: 0.1u, symbol Device:C
- added J3: Micro_SD_Card_Det1, symbol Connector:Micro_SD_Card_Det1
- added R89, R90: 0, symbol Device:R_US
- added R91, R92, R93, R94, R95, R96, R97, R98, R99: 33, symbol Device:R_US
- added U18: (no value), ST_QFN40P350X120X50-17L:PCBComponent_1, symbol stuff:EMIF06-MSD02N16
Connections:
- new net: R93.1, U18.8 (DAT1)
- new net: J3.1 (DAT2), R97.1
- new net: R90.1, U18.16 (RDAT3_UP)
- new net: R89.2, U18.2 (RDAT3_DOWN)
- new net: R94.1, U18.3 (DAT2)
- new net: R95.1, U18.4 (DAT3)
- new net: R91.1, U18.6 (CLK_IN)
- new net: R92.1, U18.7 (DAT0)
- new net: J3.7 (DAT0), R98.1
- new net: J3.2 (DAT3/CD), R96.1
- new net: J3.8 (DAT1), R99.1
- new net +3V3: C56.1, C57.1, J3.4 (VDD), R90.2, U18.15 (VCC)
- new net CLK: J3.5 (CLK), U18.11 (CLK_OUT)
- new net CMD: J3.3 (CMD), U18.12 (CMD_OUT)
- new net DAT0: R98.2, U18.10 (DAT0_OUT)
- new net DAT1: R99.2, U18.9 (DAT1_OUT)
- new net DAT2: R97.2, U18.14 (DAT2_OUT)
- new net DAT3: R96.2, U18.13 (DAT3_OUT)
- new net GND: C56.2, C57.2, J3.6 (VSS), J3.SH (SHIELD), R89.1, U18.EP (GND)
- new net SD_CLK_IN: R91.2
- new net SD_CMD_IN: U18.5 (CMD_IN)
- new net SD_DAT0: R92.2
- new net SD_DAT1: R93.2
- new net SD_DAT2: R94.2
- new net SD_DAT3: R95.2
- new net SD_Detect: J3.9 (DET), U18.1 (WP/CD)
Other:
- note added: "C57 is the SD card capacitor"
- note added: "Decoupling capacitor is on ESD protection schematic (C57)"
- note added: "R89 and R90 are card detect type selection resistors. R89 provides electrical card detect, whereas R90 provides mechanical card detect."
- note added: "SD Card"
- note added: "SD card EMI/ESD shielding"
